File: heptaphasis.brd (EAGLE design)
At the start: 100 x 45.2 mm, 121 parts, among them IC1 TL074D, IC2 TL072D, IC3 TL074D, IC4 LM13700M, T1 BC847, T2 BC847, T3 BC847, T4 BC847, T5 BC847, T6 BC847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

Commit message: Add files via upload
Parts:
- C21: value 100n -> do not install
- C24: value 1u -> 10u
- R38: value 10 -> do not install
- R39: value 100k -> do not install
- R56: value 2.2M -> 1M
- T8: value BC857 -> do not install
Changed lines of the file:
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@@
 <setting verticaltext="up"/>
 </settings>
-<grid distance="0.5" unitdist="mil" unit="mil" style="lines" multiple="1" display="yes" altdistance="1" altunitdist="mil" altunit="mil"/>
+<grid distance="5" unitdist="mil" unit="mil" style="lines" multiple="1" display="yes" altdistance="1" altunitdist="mil" altunit="mil"/>
 <layers>
-<layer number="1" name="Top" color="4" fill="1" visible="no" active="yes"/>
+<layer number="1" name="Top" color="4" fill="1" visible="yes" active="yes"/>
 <layer number="2" name="layer2" color="15" fill="1" visible="no" active="no"/>
 <layer number="3" name="layer3" color="15" fill="1" visible="no" active="no"/>
@@
 <layer number="14" name="layer14" color="15" fill="1" visible="no" active="no"/>
 <layer number="15" name="layer15" color="15" fill="1" visible="no" active="no"/>
-<layer number="16" name="Bottom" color="1" fill="1" visible="yes" active="yes"/>
+<layer number="16" name="Bottom" color="1" fill="1" visible="no" active="yes"/>
 <layer number="17" name="Pads" color="2" fill="1" visible="yes" active="yes"/>
 <layer number="18" name="Vias" color="2" fill="1" visible="yes" active="yes"/>
 <layer number="19" name="Unrouted" color="6" fill="1" visible="yes" active="yes"/>
 <layer number="20" name="Dimension" color="24" fill="1" visible="yes" active="yes"/>
-<layer number="21" name="tPlace" color="7" fill="1" visible="no" active="yes"/>
-<layer number="22" name="bPlace" color="7" fill="1" visible="yes" active="yes"/>
-<layer number="23" name="tOrigins" color="15" fill="1" visible="no" active="yes"/>
-<layer number="24" name="bOrigins" color="15" fill="1" visible="yes" active="yes"/>
-<layer number="25" name="tNames" color="7" fill="1" visible="no" active="yes"/>
-<layer number="26" name="bNames" color="7" fill="1" visible="yes" active="yes"/>
+<layer number="21" name="tPlace" color="7" fill="1" visible="yes" active="yes"/>
+<layer number="22" name="bPlace" color="7" fill="1" visible="no" active="yes"/>
+<layer number="23" name="tOrigins" color="15" fill="1" visible="yes" active="yes"/>
+<layer number="24" name="bOrigins" color="15" fill="1" visible="no" active="yes"/>
+<layer number="25" name="tNames" color="7" fill="1" visible="yes" active="yes"/>
+<layer number="26" name="bNames" color="7" fill="1" visible="no" active="yes"/>
 <layer number="27" name="tValues" color="7" fill="1" visible="no" active="yes"/>
 <layer number="28" name="bValues" color="7" fill="1" visible="no" active="yes"/>
@@
 <layer number="37" name="tTest" color="7" fill="1" visible="no" active="yes"/>
 <layer number="38" name="bTest" color="7" fill="1" visible="no" active="yes"/>
-<layer number="39" name="tKeepout" color="4" fill="11" visible="no" active="yes"/>
-<layer number="40" name="bKeepout" color="1" fill="11" visible="yes" active="yes"/>
-<layer number="41" name="tRestrict" color="4" fill="10" visible="no" active="yes"/>
-<layer number="42" name="bRestrict" color="1" fill="10" visible="yes" active="yes"/>
+<layer number="39" name="tKeepout" color="4" fill="11" visible="yes" active="yes"/>
+<layer number="40" name="bKeepout" color="1" fill="11" visible="no" active="yes"/>
+<layer number="41" name="tRestrict" color="4" fill="10" visible="yes" active="yes"/>
+<layer number="42" name="bRestrict" color="1" fill="10" visible="no" active="yes"/>
 <layer number="43" name="vRestrict" color="2" fill="10" visible="no" active="yes"/>
 <layer number="44" name="Drills" color="7" fill="1" visible="no" active="yes"/>
@@
 <layer number="49" name="Reference" color="7" fill="1" visible="no" active="yes"/>
 <layer number="50" name="dxf" color="7" fill="1" visible="no" active="no"/>
-<layer number="51" name="tDocu" color="7" fill="1" visible="no" active="yes"/>
-<layer number="52" name="bDocu" color="7" fill="1" visible="yes" active="yes"/>
+<layer number="51" name="tDocu" color="7" fill="1" visible="yes" active="yes"/>
+<layer number="52" name="bDocu" color="7" fill="1" visible="no" active="yes"/>
 <layer number="53" name="tGND_GNDA" color="7" fill="9" visible="no" active="no"/>
 <layer number="54" name="bGND_GNDA" color="1" fill="9" visible="no" active="no"/>
@@
 <layer number="132" name="test" color="7" fill="1" visible="no" active="yes"/>
 <layer number="144" name="Drill_legend" color="7" fill="1" visible="no" active="yes"/>
-<layer number="150" name="Notes" color="7" fill="1" visible="no" active="yes"/>
+<layer number="150" name="Notes" color="7" fill="1" visible="yes" active="yes"/>
 <layer number="151" name="HeatSink" color="7" fill="1" visible="no" active="yes"/>
 <layer number="152" name="_bDocu" color="7" fill="1" visible="no" active="no"/>
@@
 <text x="18.5166" y="31.2928" size="1.016" layer="25" font="vector" ratio="10" align="top-center">+</text>
 <text x="7.4422" y="31.2928" size="1.016" layer="25" font="vector" ratio="10" align="top-center">+</text>
+<dimension x1="1.905" y1="45.212" x2="68.3514" y2="45.212" x3="35.1282" y3="45.9486" textsize="0.3048" layer="150" width="0.0254" precision="4"/>
+<dimension x1="29.6672" y1="45.1612" x2="29.6672" y2="42.164" x3="26.535828125" y3="43.6626" textsize="0.8128" layer="150" width="0.0254"/>
+<dimension x1="29.591" y1="44.831" x2="27.94" y2="44.831" x3="28.7655" y3="44.45" textsize="0.8128" layer="150" width="0.0254"/>
+<dimension x1="29.591" y1="44.45" x2="31.242" y2="44.45" x3="30.4165" y3="43.561" textsize="0.8128" layer="150" width="0.0254"/>
 </plain>
 <attributes>
@@
 <attribute name="VALUE" x="26.924" y="5.842" size="1.27" layer="27" rot="R90"/>
 </element>
-<element name="C21" library="rcl" library_urn="urn:adsk.eagle:library:334" package="C0805" package3d_urn="urn:adsk.eagle:package:23617/2" value="100n" x="74.676" y="13.208" smashed="yes" rot="R270">
+<element name="C21" library="rcl" library_urn="urn:adsk.eagle:library:334" package="C0805" package3d_urn="urn:adsk.eagle:package:23617/2" value="do not install" x="74.676" y="13.208" smashed="yes" rot="R270">
 <attribute name="NAME" x="75.057" y="11.4046" size="1.016" layer="25" font="vector" rot="R180"/>
 <attribute name="SPICEPREFIX" value="C" x="2.286" y="-60.452" size="1.778" layer="27" rot="R270" display="off"/>
@@
 <attribute name="VALUE" x="87.757" y="24.384" size="1.27" layer="27"/>
 </element>
-<element name="R38" library="rcl" library_urn="urn:adsk.eagle:library:334" package="R0805" package3d_urn="urn:adsk.eagle:package:23553/2" value="10" x="74.168" y="23.368" smashed="yes" rot="R180">
+<element name="R38" library="rcl" library_urn="urn:adsk.eagle:library:334" package="R0805" package3d_urn="urn:adsk.eagle:package:23553/2" value="do not install" x="74.168" y="23.368" smashed="yes" rot="R180">
 <attribute name="NAME" x="75.3618" y="22.5552" size="1.016" layer="25" font="vector" rot="R180"/>
 <attribute name="SPICEPREFIX" value="R" x="-12.192" y="102.108" size="1.778" layer="27" rot="R180" display="off"/>
 <attribute name="VALUE" x="74.803" y="25.908" size="1.27" layer="27" rot="R180"/>
 </element>
-<element name="R39" library="rcl" library_urn="urn:adsk.eagle:library:334" package="R0805" package3d_urn="urn:adsk.eagle:package:23553/2" value="100k" x="72.644" y="18.796" smashed="yes" rot="R270">
+<element name="R39" library="rcl" library_urn="urn:adsk.eagle:library:334" package="R0805" package3d_urn="urn:adsk.eagle:package:23553/2" value="do not install" x="72.644" y="18.796" smashed="yes" rot="R270">
 <attribute name="NAME" x="70.8152" y="20.1168" size="1.016" layer="25" font="vector" rot="R270"/>
 <attribute name="SPICEPREFIX" value="R" x="6.604" y="-4.064" size="1.778" layer="27" rot="R270" display="off"/>
 <attribute name="VALUE" x="70.104" y="19.431" size="1.27" layer="27" rot="R270"/>
 </element>
-<element name="R56" library="rcl" library_urn="urn:adsk.eagle:library:334" package="R0805" package3d_urn="urn:adsk.eagle:package:23553/2" value="2.2M" x="92.964" y="11.176" smashed="yes" rot="R270">
+<element name="R56" library="rcl" library_urn="urn:adsk.eagle:library:334" package="R0805" package3d_urn="urn:adsk.eagle:package:23553/2" value="1M" x="92.964" y="11.176" smashed="yes" rot="R270">
 <attribute name="NAME" x="94.361" y="9.2202" size="1.016" layer="25" font="vector" rot="R180"/>
 <attribute name="SPICEPREFIX" value="R" x="26.924" y="-18.034" size="1.778" layer="27" rot="R270" display="off"/>
@@
 <attribute name="VALUE" x="51.094" y="28.051" size="1" layer="27" font="vector" rot="R180"/>
 </element>
-<element name="T8" library="nxp_60_sot457" package="SOT23" value="BC857" x="71.12" y="13.208" smashed="yes" rot="R180">
+<element name="T8" library="nxp_60_sot457" package="SOT23" value="do not install" x="71.12" y="13.208" smashed="yes" rot="R180">
 <attribute name="NAME" x="73.0396" y="16.2486" size="1.016" layer="25" font="vector" rot="R180"/>
 <attribute name="VALUE" x="68.62" y="14.208" size="1" layer="27" font="vector" rot="R180"/>
@@
 <attribute name="VALUE" x="53.34" y="16.891" size="1.27" layer="27" rot="R270"/>
 </element>
-<element name="C24" library="rcl" library_urn="urn:adsk.eagle:library:334" package="C0805" package3d_urn="urn:adsk.eagle:package:23617/2" value="1u" x="92.964" y="16.764" smashed="yes" rot="R270">
+<element name="C24" library="rcl" library_urn="urn:adsk.eagle:library:334" package="C0805" package3d_urn="urn:adsk.eagle:package:23617/2" value="10u" x="92.964" y="16.764" smashed="yes" rot="R270">
 <attribute name="NAME" x="94.1832" y="15.0114" size="1.016" layer="25" font="vector" rot="R180"/>
 <attribute name="SPICEPREFIX" value="C" x="92.964" y="16.764" size="1.778" layer="27" rot="R270" display="off"/>
